File: hw/ssh-bridge-for-raspberrypi.kicad_pcb (KiCad board)
At the start: 2 copper layers, 93 x 50 mm, 38 parts, among them J101 USB4105-GF-A, J102 USB4105-GF-A, J103 PinHeader Conn_01x08, J104 Conn_02x05_Odd_Even, J105 USB_A, J106 Conn_01x03, SW304 1, U101 ST7789V_TFT_DISPLAY_8P, U102 TLP3555A, U103 AZ1117-CH3.3TRG1, U201 ESP32-S3-WROOM-1-N16R8

Commit message: ssh-serrial-bridge for raspberrypi
Parts:
- removed D102: CUHS20F60, Diode_SMD:D_PowerDI-123
- removed J103: PinHeader Conn_01x08, Connector_PinHeader_2.54mm:PinHeader_1x08_P2.54mm_Vertical
- removed J106: Conn_01x03, Connector_PinHeader_2.54mm:PinHeader_1x03_P2.54mm_Vertical
- added J1: Conn_01x04, Connector_PinHeader_2.54mm:PinHeader_1x04_P2.54mm_Vertical, F.Cu at (127.0, 96.2)
- added J2: Conn_01x10, Connector_PinHeader_2.54mm:PinHeader_1x10_P2.54mm_Vertical, F.Cu at (186.5, 122.2)
Connections:
- C101 pad 1: /VBUS_IN -> +5V
- D101 pad 1: /VBUS_IN -> +5V
- J101 pad A4: /VBUS_IN -> +5V
- J101 pad A9: /VBUS_IN -> +5V
- J101 pad B4: /VBUS_IN -> +5V
- J101 pad B9: /VBUS_IN -> +5V
- R204 pad 1: /VBUS_IN -> +5V
- U102 pad 4: /VBUS_IN -> +5V
- U103 pad 3: /VBUS_IN -> +5V
Routing:
- net /VBUS_IN: track 116.3 -> 0.00 mm, vias 3 -> 0
- net +5V: track 9.31 -> 124.4 mm, vias 0 -> 3
- net +3.3V: track 92.6 -> 126.3 mm
- net GND: vias 67 -> 72
- added copper zone on F.Cu, net +5V
- removed copper zone on F.Cu, net /VBUS_IN
Other:
- board text added: "(C) 2026 HNZ"
- board text added: "3V3"
- board text added: "SSH-SERIAL BRIDGE AND VIEWER R4"
- board text removed: "(C) 2026 HNZ SSH-SERIAL BRIDGE AND VIEWER R3"
